Commit message: added new  barret hand packages including description, msgs and control (still need to clean the package). Added also some mitsubishi related missing files

File: seekur_jr_arm/terabot/terabot_description/urdf/terabot.urdf.xacro (robot description, xacro)
@@ -14,5 +14,5 @@
   <link name="arm_base_link">
     <visual>
-      <origin xyz="0 0 ${(80/2)*BASE}" rpy="0 ${-pi/2} ${pi/2}" />
+      <origin xyz="0 0 ${(80/2)*BASE}" rpy="0 ${-PI/2} ${PI/2}" />
       <geometry>
         <mesh filename="package://terabot_description/meshes/base.stl" scale="0.001 0.001 0.001"/>
