Commit message: seekur_jr related packages are now better organized. The terabot arm is now independent from the seekur_jr and the seekur_base_link was removed

File: seekur_jr/seekur_jr_description/robots/seekur_jr.urdf.xacro (robot description, xacro)
@@ -18,5 +18,6 @@
     <origin xyz="0.229108 0 0.4953"/>
   </joint>-->
-  <xacro:include filename="$(find seekur_jr_description)/urdf/seekur_jr.urdf.xacro" />
+  <xacro:include filename="$(find seekur_jr_description)/urdf/seekur_jr.xacro" />
+  <xacro:include filename="$(find seekur_jr_description)/urdf/sensors/sensors.xacro" />
   <!--<xacro:include filename="$(find seekur_jr_description)/urdf/arm/arm.urdf.xacro" />-->
   <!--<xacro:include filename="$(find seekur_jr_description)/urdf/gripper/gripper.urdf.xacro" />

File: seekur_jr/seekur_jr_description/robots/seekur_jr_with_arm.urdf.xacro (robot description, xacro)
@@ -12,12 +12,4 @@
     <origin xyz="0 0 2.0"/>
   </joint>-->
-  <!-- Joint that links the terabot-s arm to the seekur jr robot -->
-  <link name="base_link">
-  </link>
-  <joint name="base_to_seekur" type="fixed">
-    <parent link="base_link"/>
-    <child link="seekur_base_link"/>
-    <origin xyz="0 0 0"/>
-  </joint>
   <joint name="base_to_arm" type="fixed">
     <parent link="seekur_top_link"/>
@@ -25,6 +17,6 @@
     <origin xyz="0.3525 0 0"/> <!-- 0.425/2 + ~0.14 -->
   </joint>
-  <xacro:include filename="$(find seekur_jr_description)/urdf/seekur_jr.urdf.xacro" />
+  <xacro:include filename="$(find seekur_jr_description)/urdf/seekur_jr.xacro" />
   <xacro:include filename="$(find seekur_jr_description)/urdf/sensors/sensors.xacro" />
-  <xacro:include filename="$(find terabot_description)/urdf/terabot.urdf.xacro" />
+  <xacro:include filename="$(find terabot_description)/urdf/terabot.xacro" />
 </robot>

File: seekur_jr/seekur_jr_description/urdf/seekur_jr.xacro (robot description, xacro)
@@ -3,5 +3,5 @@
   <property name="pi" value="3.1415926535897931" />
   <property name="wheel_z_offset" value="0.1" />
-  <link name="seekur_base_link" >
+  <link name="base_link" >
     <visual>
       <origin xyz="0 0 0" rpy="${pi/2} 0 ${-pi/2}" />
@@ -27,5 +27,5 @@
   <joint name="seekur_base_to_top_joint" type="fixed">
       <origin xyz="0 0 0.406" rpy="0 0 0" /> <!-- 386 + 20 plaque -->
-      <parent link="seekur_base_link"/>
+      <parent link="base_link"/>
       <child link="seekur_top_link"/>
   </joint>

File: terabot/terabot_description/robots/terabot.urdf.xacro (robot description, xacro)
@@ -13,4 +13,4 @@
     <dynamics damping="0.001"/>
   </joint>
-  <xacro:include filename="$(find terabot_description)/urdf/terabot.urdf.xacro" />
+  <xacro:include filename="$(find terabot_description)/urdf/terabot.xacro" />
 </robot>

File: terabot/terabot_description/urdf/terabot.xacro (robot description, xacro)
@@ -52,4 +52,9 @@
     </visual>
     <collision>
+      <origin xyz="0 0 ${-(80/2)*BASE}" rpy="0 ${-pi/2} ${pi/2}" />
+      <geometry>
+        <mesh filename="package://terabot_description/meshes/shoulder.stl" scale="0.001 0.001 0.001"/>
+      </geometry>
+      <material name="Blue"/>
     </collision>
     <inertial>
@@ -79,4 +84,9 @@
     </visual>
     <collision>
+      <origin xyz="${-(229/2)*BASE+forearm_link_x_offset} ${-(229/2)*BASE+forearm_link_y_offset} 0" rpy="0 0 ${PI/4}" />
+      <geometry>
+        <mesh filename="package://terabot_description/meshes/forearm.stl" scale="0.001 0.001 0.001"/>
+      </geometry>
+      <material name="Blue"/>
     </collision>
     <inertial>
@@ -174,5 +184,5 @@
     </inertial>
   </link>
-  <joint name="gripper_l_finger_joint" type="fixed">
+  <!--	<joint name="gripper_l_finger_joint" type="fixed">
     <origin xyz="${gripper_l_finger_joint_x_offset} 0 0" rpy="0 -${PI/2} ${-PI/2}"/>
     <limit effort="1000.0" lower="${-170*(PI/180)}" upper="${170*(PI/180)}" velocity="0.5"/>
@@ -196,5 +206,5 @@
 	  izz="1.0"/>
     </inertial>
-  </link>
+  </link>-->
   <transmission name="tran1">
     <type>transmission_interface/SimpleTransmission</type>
