Commit message: mitsubishi arm working in gazebo with kinect sensor

File: mitsubishi_arm/mitsubishi_arm_description/robots/mitsubishi_rv_6sdl.urdf.xacro (robot description, xacro)
@@ -31,10 +31,22 @@
   <xacro:include filename="$(find mitsubishi_arm_description)/urdf/mitsubishi_rv_6sdl_arm.xacro" />
   <!-- Kinect -->
-  <xacro:include filename="$(find mitsubishi_arm_description)/urdf/sensors.xacro" />
+  <!--<xacro:include filename="$(find mitsubishi_arm_description)/urdf/sensors.xacro" />-->
   <!-- kinect to base link -->
-  <joint name="camera_in_world_joint" type="fixed">
+ <!-- <joint name="camera_in_world_joint" type="fixed">
     <parent link="base_link"/>
     <child link="camera_link"/>
     <origin xyz="0.796357 0.919602 0.431341" rpy="0.0247013 0.415733 -1.55723"/>
-  </joint>
+  </joint>  -->
+  <!-- Kinect Camera Location (Nominally 0) -->
+  <property name="cal_kinect_x" value="0.0" />
+  <property name="cal_kinect_y" value="0.0" />
+  <property name="cal_kinect_z" value="0.0" />
+  <property name="cal_kinect_roll" value="0.0" />
+  <property name="cal_kinect_pitch" value="0.0" />
+  <property name="cal_kinect_yaw" value="0.0" />
+  <xacro:include filename="$(find mitsubishi_arm_description)/urdf/sensors.urdf.xacro" />
+  <!-- Base of Kinect/Prosilica Mount -->
+  <xacro:kinect_camera_v0 name="camera" parent="base_link" >
+     <origin xyz="0.796357 0.919602 0.431341" rpy="0.0247013 0.415733 -1.55723"/>
+  </xacro:kinect_camera_v0 >
 </robot>
